Commit message: Added diff_robot model

File: ros_robot_description_pkg/urdf/seven_dof_arm.urdf (robot description, URDF)
Before this commit: robot seven_dof_arm, 12 links, 11 joints
Joints:
- joint bottom_joint: child base_link -> bottom_link; parent bottom_link -> base_link
- joint gripper_roll_joint: origin xyz=0 0 0.080 rpy=4.712384999999999 -1.570795 0 -> xyz=0 0 0.080 rpy=4.712385 -1.570795 0
